File: BusinessCardOscillator/BusinessCardOscillator.kicad_pcb (KiCad board)
At the start: 2 copper layers, 88.9 x 50.8 mm, 9 parts, among them J2 VCO_OUT, U1 NE555P, U2 NE555P

Commit message: Tried inkscape
Parts:
- added BT1: Battery, Connector_PinHeader_2.54mm:PinHeader_1x02_P2.54mm_Vertical, F.Cu at (95.0, 84.8)
- C2: value 10nF -> 100nF
- J2: value VCO_OUT -> AudioJack2_SwitchT
- moved RV2 5.34 mm to (133.6, 92.5)
Routing:
- net +9V: track 51.0 -> 0.00 mm
- net Net-(U1-Pad3): track 23.1 -> 0.00 mm
- net Net-(C1-Pad1): track 18.3 -> 0.00 mm
- net Net-(C3-Pad1): track 15.4 -> 0.00 mm
- net Net-(C2-Pad1): track 14.5 -> 0.00 mm
- net Net-(R1-Pad1): track 12.7 -> 0.00 mm
- net Net-(C3-Pad2): track 10.2 -> 0.00 mm
Other:
- net class Default removed
