File: KiCAD/SynthCard.kicad_sch (KiCad schematic)
At the start: 12 parts, among them J2 AudioJack2_SwitchT, U1 NE555P, U2 NE555P

Commit message: Added working bom
Parts:
- BT1, D1: Type (none) -> Through-hole
- C1: Manufacturers Name (none) -> KEMET; Manufacturers Part Number (none) -> MMK5103K50J01L4BULK; Part Description (none) -> Film Capacitors 50volts 0.01uF 10% LS 5mm; Type (none) -> Through-hole
- C2: Manufacturers Name (none) -> KEMET; Manufacturers Part Number (none) -> MMK5104K50J01L4BULK; Part Description (none) -> Film Capacitors 50volts 0.1uF 10% LS 5mm; Type (none) -> Through-hole
- C3: Manufacturers Name (none) -> Nichicon; Manufacturers Part Number (none) -> UVR1E100MDD1TD; Part Description (none) -> Aluminum Electrolytic Capacitors - Radial Leaded 25volts 10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; Type (none) -> Through-hole
- J2: Manufacturers Name (none) -> Tayda Electronics; Manufacturers Part Number (none) -> PJ-3001F; Type (none) -> Through-hole
- R1: Manufacturers Name (none) -> KOA Speer; Manufacturers Part Number (none) -> MF1/4DCT26A1001F; Type (none) -> Through-hole
- R2: Manufacturers Name (none) -> KOA Speer; Manufacturers Part Number (none) -> MF1/4DC1002F; Type (none) -> Through-hole
- RV1, RV2: Manufacturers Name (none) -> Alpha (Taiwan); Manufacturers Part Number (none) -> RV09AF-40-20K-B500K; Type (none) -> Through-hole
- U1, U2: Manufacturers Name (none) -> Texas Instruments; Manufacturers Part Number (none) -> NE555P; Package (none) -> PDIP-8; Part Description (none) -> Timers & Support Products; Type (none) -> Through-hole
Changed lines of the file:
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@@
+      (effects (font (size 1.27 1.27)) hide)
+    )
+    (property "Manufacturers Name" " KOA Speer" (id 4) (at 145.415 104.521 0)
+      (effects (font (size 1.27 1.27)) hide)
+    )
+    (property "Manufacturers Part Number" "MF1/4DCT26A1001F" (id 5) (at 145.415 104.521 0)
+      (effects (font (size 1.27 1.27)) hide)
+    )
+    (property "Type" "Through-hole" (id 6) (at 145.415 104.521 0)
       (effects (font (size 1.27 1.27)) hide)
     )
@@
       (effects (font (size 1.27 1.27)) hide)
     )
+    (property "Manufacturers Name" "KEMET" (id 4) (at 107.315 116.586 0)
+      (effects (font (size 1.27 1.27)) hide)
+    )
+    (property "Manufacturers Part Number" "MMK5103K50J01L4BULK" (id 5) (at 107.315 116.586 0)
+      (effects (font (size 1.27 1.27)) hide)
+    )
+    (property "Part Description" "Film Capacitors 50volts 0.01uF 10% LS 5mm" (id 6) (at 107.315 116.586 0)
+      (effects (font (size 1.27 1.27)) hide)
+    )
+    (property "Type" "Through-hole" (id 7) (at 107.315 116.586 0)
+      (effects (font (size 1.27 1.27)) hide)
+    )
     (pin "1")
     (pin "2")
@@
       (effects (font (size 1.27 1.27)) hide)
     )
+    (property "Manufacturers Name" "Alpha (Taiwan) " (id 4) (at 143.51 87.376 0)
+      (effects (font (size 1.27 1.27)) hide)
+    )
+    (property "Manufacturers Part Number" "RV09AF-40-20K-B500K" (id 5) (at 143.51 87.376 0)
+      (effects (font (size 1.27 1.27)) hide)
+    )
+    (property "Type" "Through-hole" (id 6) (at 143.51 87.376 0)
+      (effects (font (size 1.27 1.27)) hide)
+    )
     (pin "1")
     (pin "2")
@@
       (effects (font (size 1.27 1.27)) hide)
     )
+    (property "Manufacturers Name" "KEMET" (id 4) (at 193.675 116.586 0)
+      (effects (font (size 1.27 1.27)) hide)
+    )
+    (property "Manufacturers Part Number" "MMK5104K50J01L4BULK" (id 5) (at 193.675 116.586 0)
+      (effects (font (size 1.27 1.27)) hide)
+    )
+    (property "Part Description" "Film Capacitors 50volts 0.1uF 10% LS 5mm" (id 6) (at 193.675 116.586 0)
+      (effects (font (size 1.27 1.27)) hide)
+    )
+    (property "Type" "Through-hole" (id 7) (at 193.675 116.586 0)
+      (effects (font (size 1.27 1.27)) hide)
+    )
     (pin "1")
     (pin "2")
@@
     )
     (property "Datasheet" "~" (id 3) (at 193.675 87.376 0)
+      (effects (font (size 1.27 1.27)) hide)
+    )
+    (property "Manufacturers Name" "Alpha (Taiwan) " (id 4) (at 193.675 87.376 0)
+      (effects (font (size 1.27 1.27)) hide)
+    )
+    (property "Manufacturers Part Number" "RV09AF-40-20K-B500K" (id 5) (at 193.675 87.376 0)
+      (effects (font (size 1.27 1.27)) hide)
+    )
+    (property "Type" "Through-hole" (id 6) (at 193.675 87.376 0)
       (effects (font (size 1.27 1.27)) hide)
     )
@@
       (effects (font (size 1.27 1.27)) hide)
     )
+    (property "Manufacturers Name" "Nichicon" (id 4) (at 205.105 94.361 0)
+      (effects (font (size 1.27 1.27)) hide)
+    )
+    (property "Manufacturers Part Number" "UVR1E100MDD1TD" (id 5) (at 205.105 94.361 0)
+      (effects (font (size 1.27 1.27)) hide)
+    )
+    (property "Part Description" "Aluminum Electrolytic Capacitors - Radial Leaded 25volts 10uF" (id 6) (at 205.105 94.361 0)
+      (effects (font (size 1.27 1.27)) hide)
+    )
+    (property "Type" "Through-hole" (id 7) (at 205.105 94.361 0)
+      (effects (font (size 1.27 1.27)) hide)
+    )
     (pin "1")
     (pin "2")
@@
     )
     (property "Datasheet" "~" (id 3) (at 220.98 94.361 0)
+      (effects (font (size 1.27 1.27)) hide)
+    )
+    (property "Manufacturers Name" "Tayda Electronics" (id 4) (at 220.98 94.361 0)
+      (effects (font (size 1.27 1.27)) hide)
+    )
+    (property "Manufacturers Part Number" "PJ-3001F" (id 5) (at 220.98 94.361 0)
+      (effects (font (size 1.27 1.27)) hide)
+    )
+    (property "Type" "Through-hole" (id 6) (at 220.98 94.361 0)
       (effects (font (size 1.27 1.27)) hide)
     )
@@
     )
     (property "Datasheet" "http://www.ti.com/lit/ds/symlink/ne555.pdf" (id 3) (at 147.955 109.601 0)
+      (effects (font (size 1.27 1.27)) hide)
+    )
+    (property "Manufacturers Name" "Texas Instruments" (id 4) (at 126.365 99.441 0)
+      (effects (font (size 1.27 1.27)) hide)
+    )
+    (property "Manufacturers Part Number" "NE555P" (id 5) (at 126.365 99.441 0)
+      (effects (font (size 1.27 1.27)) hide)
+    )
+    (property "Package" "PDIP-8" (id 6) (at 126.365 99.441 0)
+      (effects (font (size 1.27 1.27)) hide)
+    )
+    (property "Part Description" "Timers & Support Products " (id 7) (at 126.365 99.441 0)
+      (effects (font (size 1.27 1.27)) hide)
+    )
+    (property "Type" "Through-hole" (id 8) (at 126.365 99.441 0)
       (effects (font (size 1.27 1.27)) hide)
     )
@@
       (effects (font (size 1.27 1.27)) hide)
     )
+    (property "Manufacturers Name" "Texas Instruments" (id 4) (at 176.53 99.441 0)
+      (effects (font (size 1.27 1.27)) hide)
+    )
+    (property "Manufacturers Part Number" "NE555P" (id 5) (at 176.53 99.441 0)
+      (effects (font (size 1.27 1.27)) hide)
+    )
+    (property "Package" "PDIP-8" (id 6) (at 176.53 99.441 0)
+      (effects (font (size 1.27 1.27)) hide)
+    )
+    (property "Part Description" "Timers & Support Products " (id 7) (at 176.53 99.441 0)
+      (effects (font (size 1.27 1.27)) hide)
+    )
+    (property "Type" "Through-hole" (id 8) (at 176.53 99.441 0)
+      (effects (font (size 1.27 1.27)) hide)
+    )
     (pin "1")
     (pin "8")
@@
       (effects (font (size 1.27 1.27)) hide)
     )
+    (property "Type" "Through-hole" (id 4) (at 95.885 101.981 0)
+      (effects (font (size 1.27 1.27)) hide)
+    )
     (pin "1")
     (pin "2")
@@
       (effects (font (size 1.27 1.27)) hide)
     )
+    (property "Manufacturers Name" " KOA Speer" (id 4) (at 89.027 79.121 0)
+      (effects (font (size 1.27 1.27)) hide)
+    )
+    (property "Manufacturers Part Number" "MF1/4DC1002F" (id 5) (at 89.027 79.121 0)
+      (effects (font (size 1.27 1.27)) hide)
+    )
+    (property "Type" "Through-hole" (id 6) (at 89.027 79.121 0)
+      (effects (font (size 1.27 1.27)) hide)
+    )
     (pin "1")
     (pin "2")
@@
       (effects (font (size 1.27 1.27)) hide)
     )
+    (property "Type" "Through-hole" (id 4) (at 83.058 84.836 0)
+      (effects (font (size 1.27 1.27)) hide)
+    )
